File: hw/chibi/chibi_2024/chibi_2024.kicad_pcb (KiCad board)
At the start: 2 copper layers, 114 parts, among them P1 VIN, P2 CONN_02X05, P3 GND, P4 CONN_02X05, P5 SWD, Q1 AO3415A, Q10 Q_NPN_CBE, Q11 Q_NPN_CBE, Q2 AO3415A, Q3 AO3415A, Q4 AO3415A, Q5 AO3415A, Q6 AO3415A, Q7 AO3415A, Q8 AO3415A, Q9 Q_PNP_CBE, SW1 USER, SW2 RESET, U1 LD1117S33CTR, U2 SP3485CN, U3 STM32F030F4Px, U4 LM358, U5 74HC595_mine, U6 LM393, U7 74HC595_mine, U8 MBI5026, U9 MBI5026, Y1 8MHz

Commit message: Foo
Parts:
- removed C21, C22, C23, C24, C25, C26, C27: 100n, Capacitors_SMD:C_0603_HandSoldering
- removed D5, D6: BAR 43C, TO_SOT_Packages_SMD:SOT-23_Handsoldering
- removed P2: CONN_02X05, Pin_Headers:Pin_Header_Straight_2x05
- removed R26, R27, R28, R30: 10k, Resistors_SMD:R_0805
- removed R31: 4k7, Resistors_SMD:R_0805
- D2: footprint Diodes_SMD:SOD-323 -> Diodes_SMD:MiniMELF_Standard
- D3, D4: value BAR 43C -> D_Small; footprint TO_SOT_Packages_SMD:SOT-23_Handsoldering -> Diodes_SMD:MiniMELF_Standard
- R21: value 10k -> 470k
- R22: value 10k -> 100k
- R25, R29, R32, R33, R34, R35: footprint Resistors_SMD:R_0805 -> Resistors_SMD:R_0603_HandSoldering
- U8, U9: moved to B.Cu
- moved R15 196.7 mm to (79.4, 109.1), turned to 180 degrees
- moved R9 188.0 mm to (96.8, 97.7)
- moved R16 185.1 mm to (83.9, 101.7), turned to 270 degrees
- moved R17 185.0 mm to (97.3, 106.2), turned to 180 degrees
- moved R6 178.4 mm to (101.5, 94.6), turned to 180 degrees
- moved C8 177.0 mm to (64.8, 137.6)
- moved C2 177.0 mm to (57.0, 144.0)
- moved C6 177.0 mm to (49.5, 150.3)
- moved C7 177.0 mm to (53.7, 150.3)
- moved R22 176.1 mm to (90.9, 94.9)
- moved C18 174.7 mm to (92.8, 106.7)
- moved R23 172.8 mm to (83.9, 87.9), turned to 90 degrees
- moved R20 172.5 mm to (96.5, 86.1), turned to 90 degrees
- moved C14 171.1 mm to (101.5, 96.5), turned to 180 degrees
- moved C17 171.0 mm to (86.0, 101.4), turned to 270 degrees
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Connections:
- net /WD_REF renamed /WD_REF1
- net Net-(F1-Pad1) renamed /VDD_PRE_FUSE
- C20 pad 1: /WD_DC_A -> /WD_COMP
- D10 pad 1: /mux_mod_right/SEG_E -> /SEG_E_COM
- D10 pad 10: /mux_mod_right/SEG_F -> /SEG_F_COM
- D10 pad 11: /mux_mod_right/SEG_A -> /SEG_A_COM
- D10 pad 2: /mux_mod_right/SEG_D -> /SEG_D_COM
- D10 pad 3: /mux_mod_right/SEG_DP -> /SEG_DP_COM
- D10 pad 4: /mux_mod_right/SEG_C -> /SEG_C_COM
- D10 pad 5: /mux_mod_right/SEG_G -> /SEG_G_COM
- D10 pad 7: /mux_mod_right/SEG_B -> /SEG_B_COM
- D11 pad 1: /mux_mod_right/SEG_E -> /SEG_E_COM
- D11 pad 10: /mux_mod_right/SEG_F -> /SEG_F_COM
- D11 pad 11: /mux_mod_right/SEG_A -> /SEG_A_COM
- D11 pad 2: /mux_mod_right/SEG_D -> /SEG_D_COM
- D11 pad 3: /mux_mod_right/SEG_DP -> /SEG_DP_COM
- D11 pad 4: /mux_mod_right/SEG_C -> /SEG_C_COM
- D11 pad 5: /mux_mod_right/SEG_G -> /SEG_G_COM
- D11 pad 7: /mux_mod_right/SEG_B -> /SEG_B_COM
- D12 pad 1: /mux_mod_right/SEG_E -> /SEG_E_COM
- D12 pad 10: /mux_mod_right/SEG_F -> /SEG_F_COM
- D12 pad 11: /mux_mod_right/SEG_A -> /SEG_A_COM
- D12 pad 2: /mux_mod_right/SEG_D -> /SEG_D_COM
- D12 pad 3: /mux_mod_right/SEG_DP -> /SEG_DP_COM
- D12 pad 4: /mux_mod_right/SEG_C -> /SEG_C_COM
- D12 pad 5: /mux_mod_right/SEG_G -> /SEG_G_COM
- D12 pad 7: /mux_mod_right/SEG_B -> /SEG_B_COM
- D13 pad 1: /mux_mod_right/SEG_E -> /SEG_E_COM
- D13 pad 10: /mux_mod_right/SEG_F -> /SEG_F_COM
- D13 pad 11: /mux_mod_right/SEG_A -> /SEG_A_COM
- D13 pad 2: /mux_mod_right/SEG_D -> /SEG_D_COM
- D13 pad 3: /mux_mod_right/SEG_DP -> /SEG_DP_COM
- D13 pad 4: /mux_mod_right/SEG_C -> /SEG_C_COM
- D13 pad 5: /mux_mod_right/SEG_G -> /SEG_G_COM
- D13 pad 7: /mux_mod_right/SEG_B -> /SEG_B_COM
- D3 pad 1: /WD_DC_B -> /~WD_RST1
- D3 pad 2: /WD_DC_A -> /~WD_RST
- D4 pad 1: /WD_DC_D -> /~WD_RST2
- D4 pad 2: /WD_DC_C -> /~WD_RST
- D7 pad 1: Net-(D7-Pad1) -> GND
- D7 pad 2: /LED_ID -> Net-(D7-Pad2)
- D8 pad 1: Net-(D8-Pad1) -> GND
- D8 pad 2: /LED_ERROR -> Net-(D8-Pad2)
- D9 pad 1: Net-(D9-Pad1) -> GND
- D9 pad 2: /LED_COMM -> Net-(D9-Pad2)
- P4 pad 1: /RS485_A -> GND
- P4 pad 3: /RS485_B -> GND
- P4 pad 5: GND -> /RS485_B
- P4 pad 7: GND -> /RS485_A
- Q1 pad 1: /SEG_A_CTRL -> /SEG_C_CTRL
- Q1 pad 2: /SEG_A_COM -> /SEG_C_COM
- Q10 pad 1: /mux_mod_right/R_SET_0 -> /mux_mod_left/R_SET_0
- Q11 pad 1: /mux_mod_right/R_SET_1 -> /mux_mod_left/R_SET_1
- Q2 pad 1: /SEG_B_CTRL -> /SEG_G_CTLR
- Q2 pad 2: /SEG_B_COM -> /SEG_G_COM
- Q3 pad 1: /SEG_C_CTRL -> /SEG_B_CTRL
- Q3 pad 2: /SEG_C_COM -> /SEG_B_COM
- Q4 pad 1: /SEG_D_CTRL -> /SEG_DP_CTRL
- Q4 pad 2: /SEG_D_COM -> /SEG_DP_COM
- Q5 pad 1: /SEG_E_CTRL -> /SEG_F_CTRL
- Q5 pad 2: /SEG_E_COM -> /SEG_F_COM
- Q6 pad 1: /SEG_F_CTRL -> /SEG_D_CTRL
- Q6 pad 2: /SEG_F_COM -> /SEG_D_COM
- Q7 pad 1: /SEG_G_CTLR -> /SEG_A_CTRL
- Q7 pad 2: /SEG_G_COM -> /SEG_A_COM
- Q8 pad 1: /SEG_DP_CTRL -> /SEG_E_CTRL
- Q8 pad 2: /SEG_DP_COM -> /SEG_E_COM
- R21 pad 1: /WD_DC_A -> /WD_REF2
- R21 pad 2: /SEG_A_CTRL -> /~WD_RST2
- R22 pad 1: /WD_DC_B -> /WD_REF2
- R22 pad 2: /SEG_B_CTRL -> +3V3
- R23 pad 2: /~WD_RST -> /~WD_RST1
- R24 pad 1: /WD_DC_C -> GND
- R24 pad 2: /SEG_C_CTRL -> /WD_REF2
- R32 pad 1: GND -> /WD_COMP
- R32 pad 2: /WD_COMP -> /SEG_B_CTRL
- R35 pad 1: Net-(D7-Pad1) -> /LED_ID
- R35 pad 2: GND -> Net-(D7-Pad2)
- R36 pad 1: Net-(D8-Pad1) -> /LED_ERROR
- R36 pad 2: GND -> Net-(D8-Pad2)
- R37 pad 1: Net-(D9-Pad1) -> /LED_COMM
- R37 pad 2: GND -> Net-(D9-Pad2)
- R38 pad 1: /mux_mod_right/R_SET_0 -> /mux_mod_left/R_SET_0
- R39 pad 1: /mux_mod_right/R_SET_1 -> /mux_mod_left/R_SET_1
- U5 pad 1: /R_SET_CTRL1 -> /LED_ERROR
- U5 pad 15: /R_SET_CTRL0 -> Net-(U5-Pad15)
- U5 pad 2: Net-(U5-Pad2) -> /LED_COMM
- U5 pad 3: Net-(U5-Pad3) -> /LED_ID
- U5 pad 5: /LED_COMM -> Net-(U5-Pad5)
- U5 pad 6: /LED_ERROR -> /R_SET_CTRL0
- U5 pad 7: /LED_ID -> /R_SET_CTRL1
- U6 pad 1: /~WD_RST -> /~WD_RST1
- U6 pad 5: (no net) -> /WD_REF2
- U6 pad 6: (no net) -> /WD_COMP
- U6 pad 7: (no net) -> /~WD_RST2
- U7 pad 1: /SEG_B_CTRL -> /SEG_E_CTRL
- U7 pad 15: /SEG_A_CTRL -> /SEG_D_CTRL
- U7 pad 2: /SEG_C_CTRL -> /SEG_DP_CTRL
- U7 pad 3: /SEG_D_CTRL -> /SEG_C_CTRL
- U7 pad 4: /SEG_E_CTRL -> /SEG_G_CTLR
- U7 pad 5: /SEG_F_CTRL -> /SEG_A_CTRL
- U7 pad 6: /SEG_G_CTLR -> /SEG_B_CTRL
- U7 pad 7: /SEG_DP_CTRL -> /SEG_F_CTRL
- U8 pad 10: Net-(D11-Pad8) -> Net-(D12-Pad9)
- U8 pad 11: Net-(D11-Pad9) -> Net-(D12-Pad8)
- U8 pad 12: Net-(D11-Pad12) -> Net-(D12-Pad6)
- U8 pad 13: Net-(D12-Pad6) -> Net-(D11-Pad12)
- U8 pad 14: Net-(D12-Pad8) -> Net-(D11-Pad9)
- U8 pad 15: Net-(D12-Pad9) -> Net-(D11-Pad8)
- U8 pad 16: Net-(D12-Pad12) -> Net-(D11-Pad6)
- U8 pad 17: Net-(D13-Pad6) -> Net-(D10-Pad12)
- U8 pad 18: Net-(D13-Pad8) -> Net-(D10-Pad9)
- U8 pad 19: Net-(D13-Pad9) -> Net-(D10-Pad8)
- U8 pad 20: Net-(D13-Pad12) -> Net-(D10-Pad6)
- U8 pad 3: /mux_mod_right/CLK -> /SCK
- U8 pad 5: Net-(D10-Pad6) -> Net-(D13-Pad12)
- U8 pad 6: Net-(D10-Pad8) -> Net-(D13-Pad9)
- U8 pad 7: Net-(D10-Pad9) -> Net-(D13-Pad8)
- U8 pad 8: Net-(D10-Pad12) -> Net-(D13-Pad6)
- U8 pad 9: Net-(D11-Pad6) -> Net-(D12-Pad12)
- U9 pad 1: /mux_mod_left/GND -> GND
- U9 pad 10: Net-(D15-Pad8) -> Net-(D16-Pad9)
- U9 pad 11: Net-(D15-Pad9) -> Net-(D16-Pad8)
- U9 pad 12: Net-(D15-Pad12) -> Net-(D16-Pad6)
- U9 pad 13: Net-(D16-Pad6) -> Net-(D15-Pad12)
- U9 pad 14: Net-(D16-Pad8) -> Net-(D15-Pad9)
- U9 pad 15: Net-(D16-Pad9) -> Net-(D15-Pad8)
- U9 pad 16: Net-(D16-Pad12) -> Net-(D15-Pad6)
- U9 pad 17: Net-(D17-Pad6) -> Net-(D14-Pad12)
- U9 pad 18: Net-(D17-Pad8) -> Net-(D14-Pad9)
- U9 pad 19: Net-(D17-Pad9) -> Net-(D14-Pad8)
- U9 pad 20: Net-(D17-Pad12) -> Net-(D14-Pad6)
- U9 pad 21: /mux_mod_left/~OE -> /~OE
- U9 pad 3: /mux_mod_left/CLK -> /SCK
- U9 pad 4: /mux_mod_left/LE -> /STROBE
- U9 pad 5: Net-(D14-Pad6) -> Net-(D17-Pad12)
- U9 pad 6: Net-(D14-Pad8) -> Net-(D17-Pad9)
- U9 pad 7: Net-(D14-Pad9) -> Net-(D17-Pad8)
- U9 pad 8: Net-(D14-Pad12) -> Net-(D17-Pad6)
- U9 pad 9: Net-(D15-Pad6) -> Net-(D16-Pad12)
Routing:
- net /SEG_E_COM: track 45.1 -> 340.3 mm, vias 3 -> 9
- net /SEG_D_COM: track 48.1 -> 343.1 mm, vias 2 -> 8
- net /SEG_DP_COM: track 49.1 -> 331.5 mm, vias 2 -> 8
- net /SEG_C_COM: track 52.6 -> 320.1 mm, vias 2 -> 9
- net /SEG_G_COM: track 56.3 -> 313.8 mm, vias 2 -> 8
- net /SEG_A_COM: track 37.4 -> 292.5 mm, vias 2 -> 8
- net /SEG_F_COM: track 41.0 -> 282.3 mm, vias 2 -> 9
- net /SEG_B_COM: track 54.9 -> 272.7 mm, vias 2 -> 4
- net /SEG_COM_MEAS: track 0.00 -> 86.5 mm
- net /SEG_B_CTRL: track 0.00 -> 77.9 mm, vias 0 -> 2
- net /SEG_F_CTRL: track 0.00 -> 64.1 mm
- net Net-(D10-Pad8): track 0.00 -> 62.1 mm, vias 0 -> 2
- net Net-(D17-Pad12): track 0.00 -> 58.9 mm, vias 0 -> 2
- net Net-(D10-Pad9): track 0.00 -> 57.8 mm, vias 0 -> 2
- net /SEG_A_CTRL: track 0.00 -> 51.3 mm
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- added copper zone on F.Cu, net /VDD_PRE_FUSE
Other:
- net class moar_pwr added: clearance 0.2, trace_width 2, via_dia 0.6, via_drill 0.4

Commit message: Layout mostly done
Parts:
- added REF**: MountingHole_4.3mm_M4, Mounting_Holes:MountingHole_4.3mm_M4, F.Cu at (51.6, 47.1)
- added REF**: MountingHole_4.3mm_M4, Mounting_Holes:MountingHole_4.3mm_M4, F.Cu at (52.0, 117.5)
- added svg2mod: G***, footprints:label_comm_04, F.Cu at (139.7, 95.2)
- added svg2mod: G***, footprints:label_error_04, F.Cu at (139.7, 88.9)
- added svg2mod: G***, footprints:label_id_04, F.Cu at (139.7, 101.6)
- added svg2mod: G***, footprints:label_plus_04, F.Cu at (133.3, 53.3)
- added svg2mod: G***, footprints:label_gnd_04, F.Cu at (136.3, 117.3)
- added svg2mod: G***, footprints:label_fuse_04, F.Cu at (99.2, 119.3)
- C19, C3: footprint Capacitors_ThroughHole:C_Radial_D10_L20_P5-7.5 -> Capacitors_ThroughHole:C_Radial_D10_L20_P5
- D1: footprint Discret:D5 -> Discret:D3
- SW1, SW2: footprint Buttons_Switches_ThroughHole:SW_PUSH_SMALL -> Buttons_Switches_SMD:SW_SPST_FSMSM
- moved C6 113.7 mm to (105.7, 51.5), turned to 180 degrees
- moved C2 83.1 mm to (85.6, 66.0), turned to 180 degrees
- moved C5 81.7 mm to (102.9, 63.0)
- moved C3 78.3 mm to (115.3, 110.1), turned to 270 degrees
- moved C8 77.9 mm to (99.8, 68.0)
- moved D1 74.2 mm to (112.6, 113.7), turned to 90 degrees
- moved R1 73.6 mm to (73.0, 54.5), turned to 180 degrees
- moved C7 60.7 mm to (97.2, 108.0)
- moved C9 53.8 mm to (115.1, 99.7), turned to 270 degrees
- moved SW2 45.6 mm to (78.8, 51.5), turned to 180 degrees
- moved C1 36.8 mm to (136.9, 64.9), turned to 180 degrees
- moved SW1 31.5 mm to (139.7, 60.2), turned to 180 degrees
- moved C19 25.3 mm to (50.9, 96.0)
- moved R2 25.2 mm to (136.7, 55.5), turned to 180 degrees
- moved R36 5.12 mm to (148.0, 88.9), turned to 270 degrees
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Connections:
- U7 pad 10: VDD -> +3V3
Routing:
- net GND: track 4.41 -> 901.6 mm, vias 0 -> 74
- net +3V3: track 7.06 -> 214.9 mm, vias 0 -> 6
- net VDD: track 16.3 -> 118.4 mm, vias 0 -> 4
- net /USER_BTN: track 0.00 -> 87.2 mm, vias 0 -> 2
- net /STROBE: track 0.00 -> 71.7 mm, vias 0 -> 3
- net /CMEAS_OFFX_COMP: track 0.00 -> 69.9 mm, vias 0 -> 4
- net /CMEAS_OUT: track 0.00 -> 66.0 mm, vias 0 -> 2
- net /~OE: track 20.6 -> 82.5 mm, vias 1 -> 4
- net /AUX_STROBE: track 35.2 -> 95.9 mm, vias 0 -> 2
- net /MOSI_C0: track 0.00 -> 56.7 mm, vias 0 -> 3
- net /RST: track 0.00 -> 51.9 mm, vias 0 -> 3
- net /SEG_COM_MEAS: track 86.5 -> 137.8 mm
- net /RS485_DE: track 0.00 -> 41.1 mm
- net /RS485_TX: track 0.00 -> 28.7 mm
- net /SCK: track 45.4 -> 73.7 mm, vias 3 -> 5
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- added copper zone on B.Cu, net GND
- added copper zone on F.Cu, net GND
Other:
- board outline added: 101.6 x 78.2 mm
- net class fuck_kicad: trace_width 1 -> 0.8

Commit message: Design mostly done
Parts:
- added P2: VIN, footprints:spade_6.35mm, F.Cu at (127.0, 114.2)
- added P6: GND, footprints:spade_6.35mm, F.Cu at (127.0, 94.5)
- added svg2mod: G***, footprints:label_gnd_04, F.Cu at (127.0, 90.0)
- added svg2mod: G***, footprints:label_data_v01, F.Cu at (71.8, 93.0)
- added svg2mod: G***, footprints:megumin, B.Cu at (100.8, 77.0)
- D10, D11, D12, D13, D14, D15, D16, D17: footprint Displays_7-Segment:Cx56-12 -> footprints:7seg_4digit_cc_modified
- U8, U9: footprint footprints:SSOP24-1.0 -> footprints:SSOP24-1.0-nosilk
- moved svg2mod 69.1 mm to (136.0, 48.2)
- moved svg2mod 60.2 mm to (136.2, 113.5), turned to 270 degrees
- moved R2 6.52 mm to (143.1, 56.6)
- moved C3 5.05 mm to (119.2, 113.2), turned to 202.5 degrees
Connections:
- C3 pad 1: VDD -> /VDD_PRE_FUSE
Routing:
- net GND: track 901.6 -> 972.2 mm, vias 74 -> 79
- net /VDD_PRE_FUSE: track 68.0 -> 84.4 mm
- net /SEG_E_COM: track 340.6 -> 327.4 mm
- net /SEG_D_COM: track 341.3 -> 329.8 mm
- net /SEG_DP_COM: track 331.5 -> 321.4 mm
- net /SEG_C_COM: track 320.1 -> 311.3 mm
- net /SEG_G_COM: track 313.8 -> 306.2 mm
- net /USER_BTN: track 87.2 -> 92.1 mm
- net /RS485_DE: track 41.1 -> 42.1 mm
- net /SEG_A_CTRL: track 62.8 -> 61.9 mm

Commit message: Release v0.2
Parts:
- removed the REF** at (51.6, 47.1)
- removed the REF** at (52.0, 117.5)
- added REF**: m3_pillar, footprints:m3_pillar, F.Cu at (52.8, 48.2)
- added REF**: m3_pillar, footprints:m3_pillar, F.Cu at (52.8, 117.5)
- added svg2mod: G***, footprints:label_gnd_04, F.Cu at (61.7, 48.2)
- added svg2mod: G***, footprints:label_plus_04, F.Cu at (64.4, 113.8)
- P1, P3: footprint Mounting_Holes:MountingHole_4.3mm_M4_Pad_Via -> footprints:m3_pillar
- moved svg2mod 21.0 mm to (67.4, 72.5)
- moved Q5 4.62 mm to (54.8, 105.9), turned to 0 degrees
- moved svg2mod 0.30 mm to (136.1, 113.7)
Routing:
- net GND: track 972.2 -> 1051.5 mm, vias 79 -> 87
- net /SEG_A_CTRL: track 61.9 -> 70.0 mm
- net /SEG_DP_COM: track 321.4 -> 313.5 mm
- net /SEG_G_COM: track 306.2 -> 300.3 mm
- net /SEG_C_COM: track 311.3 -> 306.0 mm
- net /SEG_D_COM: track 329.8 -> 325.8 mm, vias 9 -> 8
- net (no net): track 0.00 -> 3.77 mm, vias 0 -> 1
- net /STROBE: track 71.7 -> 74.6 mm
- net /SCK: track 73.7 -> 76.5 mm
- net /SEG_F_COM: track 282.3 -> 284.3 mm
- net Net-(D13-Pad12): track 16.1 -> 17.8 mm
- net /SEG_E_CTRL: track 40.8 -> 42.5 mm
- net Net-(D13-Pad9): track 22.6 -> 24.1 mm
- net /SEG_B_CTRL: track 76.6 -> 78.0 mm
- net Net-(D13-Pad8): track 24.3 -> 25.7 mm
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
Commit message: foo
Other:
- board size 101.6 x 78.2 mm -> 100 x 78 mm
Changed lines of the file:
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@@
     (links 308)
     (no_connects 0)
-    (area 45.401999 39.515396 153.957624 125.872685)
+    (area 48.184999 43.612999 149.935001 121.995001)
     (thickness 1.6)
     (drawings 6)
@@
       (net 99 /mux_mod_left/VDD))
   )
+  (gr_line (start 149 121.75) (end 149 43.75) (angle 90) (layer Edge.Cuts) (width 0.15))
+  (gr_line (start 149 43.75) (end 49 43.75) (angle 90) (layer Edge.Cuts) (width 0.15))
+  (gr_line (start 49 121.75) (end 149 121.75) (angle 90) (layer Edge.Cuts) (width 0.15))
+  (gr_line (start 49 43.75) (end 49 121.75) (angle 90) (layer Edge.Cuts) (width 0.15))
   (gr_line (start 84.5 99.25) (end 82.75 99.25) (angle 90) (layer F.SilkS) (width 0.2))
-  (gr_line (start 48.26 121.92) (end 48.26 43.688) (angle 90) (layer Edge.Cuts) (width 0.15))
-  (gr_line (start 149.86 121.92) (end 48.26 121.92) (angle 90) (layer Edge.Cuts) (width 0.15))
-  (gr_line (start 149.86 43.688) (end 149.86 121.92) (angle 90) (layer Edge.Cuts) (width 0.15))
-  (gr_line (start 48.26 43.688) (end 149.86 43.688) (angle 90) (layer Edge.Cuts) (width 0.15))
   (gr_line (start 84.455 99.187) (end 85.09 99.822) (angle 90) (layer F.SilkS) (width 0.2))
   (segment (start 67.299998 49.549998) (end 68.25 49.549998) (width 1) (layer F.Cu) (net 0))
@@
   (segment (start 57.9115 73.4235) (end 59.0545 72.2805) (width 0.254) (layer F.Cu) (net 3))
   (segment (start 59.0545 72.2805) (end 60.8325 72.2805) (width 0.254) (layer F.Cu) (net 3))
-  (segment (start 52.75 48.25) (end 49.974 51.026) (width 0.254) (layer F.Cu) (net 3))
-  (segment (start 49.974 51.026) (end 49.974 53.548) (width 0.254) (layer F.Cu) (net 3))
+  (segment (start 52.75 48.25) (end 49.974 51.026) (width 0.254) (layer F.Cu) (net 3) (status 30))
+  (segment (start 49.974 51.026) (end 49.974 53.548) (width 0.254) (layer F.Cu) (net 3) (status 10))
   (via (at 52.895 53.548) (size 1) (drill 0.8) (layers F.Cu B.Cu) (net 3))
   (segment (start 51.752 54.691) (end 52.895 53.548) (width 0.254) (layer F.Cu) (net 3))
@@
   (segment (start 147.637 53.548) (end 145.097 53.548) (width 0.254) (layer B.Cu) (net 3))
   (via (at 147.637 53.548) (size 1) (drill 0.8) (layers F.Cu B.Cu) (net 3))
-  (segment (start 52.75 48.25) (end 55.453 45.547) (width 0.254) (layer F.Cu) (net 3))
+  (segment (start 52.75 48.25) (end 55.453 45.547) (width 0.254) (layer F.Cu) (net 3) (status 30))
   (segment (start 49.9745 111.206) (end 50.736 111.206) (width 0.254) (layer F.Cu) (net 3))
   (segment (start 58.61 120.985) (end 58.61 120.8405) (width 0.254) (layer F.Cu) (net 3))
@@
   (segment (start 52.133 112.603) (end 54.8 112.603) (width 0.254) (layer F.Cu) (net 3))
   (segment (start 50.736 111.206) (end 52.133 112.603) (width 0.254) (layer F.Cu) (net 3))
-  (segment (start 50.038 50.962) (end 50.038 78.486) (width 1) (layer B.Cu) (net 3))
+  (segment (start 50.038 50.962) (end 50.038 78.486) (width 1) (layer B.Cu) (net 3) (status 10))
   (via (at 50.038 85.598) (size 1) (drill 0.8) (layers F.Cu B.Cu) (net 3))
   (segment (start 50.038 83.312) (end 50.038 85.598) (width 0.254) (layer F.Cu) (net 3))
@@
   (segment (start 50.038 78.486) (end 50.038 81.026) (width 0.254) (layer F.Cu) (net 3))
   (via (at 50.038 78.486) (size 1) (drill 0.8) (layers F.Cu B.Cu) (net 3))
-  (segment (start 50.038 50.962) (end 52.75 48.25) (width 1) (layer B.Cu) (net 3))
+  (segment (start 50.038 50.962) (end 52.75 48.25) (width 1) (layer B.Cu) (net 3) (status 30))
   (segment (start 50.038 85.598) (end 50.927 86.487) (width 0.25) (layer B.Cu) (net 3))
   (segment (start 50.927 86.487) (end 50.927 91.012) (width 0.25) (layer B.Cu) (net 3))
