File: hw/chibi/chibi_2024/chibi_2024.sch (KiCad schematic (older format))
At the start: 68 parts, among them P1 VIN, P2 VIN, P3 GND, P4 CONN_02X03, P5 SWD, P6 GND, Q1 AO3415A, Q14 Q_PNP_BEC, Q15 Q_NPN_BEC, Q16 Q_NPN_BEC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

Commit message: Fixes for second prototype (v0.3)
Parts:
- D7, D8, D9: symbol LED -> LED-RESCUE-chibi_2024
Connections:
- net labels added: +5V
- wire segments 218 -> 209
Other:
- moved on the sheet: C1, C10, C2, C4, C5, C6, C7, C8, C9, U1
