File: hw/chibi/layouttest/chibi_2024.sch (KiCad schematic (older format))
At the start: 50 parts, among them P1 VIN, P3 GND, P4 CONN_02X03, P5 SWD, Q1 AO3415A, Q15 Q_NPN_BEC, Q16 Q_NPN_BEC, Q2 AO3415A, Q3 AO3415A, Q4 AO3415A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

Commit message: Add local changes
Parts:
- added C20: 100n, Capacitors_SMD:C_0603_HandSoldering, symbol C
- added D2, D3, D4: D_Small, Diodes_SMD:MiniMELF_Standard, symbol D_Small
- added JP1: rpos, footprints:solder_jumper_3mm, symbol Jumper_NC_Small
- added JP2: rneg, footprints:solder_jumper_3mm, symbol Jumper_NC_Small
- added JP3: lpos, footprints:solder_jumper_3mm, symbol Jumper_NC_Small
- added JP4: lneg, footprints:solder_jumper_3mm, symbol Jumper_NC_Small
- added P2, P6: SUP, footprints:m3_pillar, symbol CONN_01X01
- added Q14: Q_PNP_BEC, TO_SOT_Packages_SMD:SOT-23_Handsoldering, symbol Q_PNP_BEC
- added R1, R20, R25, R29: 47k, Resistors_SMD:R_0603_HandSoldering, symbol R
- added R19, R24: 10k, Resistors_SMD:R_0603_HandSoldering, symbol R
- added R21, R23: 470k, Resistors_SMD:R_0603_HandSoldering, symbol R
- added R22, R32: 100k, Resistors_SMD:R_0603_HandSoldering, symbol R
- added U6: LM393, Housings_SOIC:SOIC-8_3.9x4.9mm_Pitch1.27mm, symbol LM393
- C1, C11, C12, C13, C2, C4, C5, C6, C7, C8, C9: symbol chibi_2024-rescue:C -> C
- C10, C19, C3: symbol chibi_2024-rescue:CP -> CP
- D1: symbol chibi_2024-rescue:ZENERsmall -> D_Zener_Small
- D7, D8, D9: symbol chibi_2024-rescue:LED-RESCUE-chibi_2024 -> LED-RESCUE-chibi_2024
- F1: footprint Fuse_Holders_and_Fuses:Fuseholder5x20_horiz_open_universal_Type-III -> Fuse_Holders_and_Fuses:Fuseholder5x20_horiz_open_inline_Type-I; symbol chibi_2024-rescue:F_Small -> Fuse_Small
- P1: value VIN -> SUP; symbol chibi_2024-rescue:CONN_01X01 -> CONN_01X01
- P3: value GND -> SUP; symbol chibi_2024-rescue:CONN_01X01 -> CONN_01X01
- P4: symbol chibi_2024-rescue:CONN_02X03 -> CONN_02X03
- P5: symbol chibi_2024-rescue:CONN_01X04 -> CONN_01X04
- Q1, Q2, Q3, Q4, Q5, Q6, Q7, Q8: symbol chibi_2024-rescue:Q_PMOS_GSD -> Q_PMOS_GSD
- Q15, Q16: symbol chibi_2024-rescue:Q_NPN_BEC -> Q_NPN_BEC
- R3, R33, R34, R35, R36, R37, R4, R44, R5: symbol chibi_2024-rescue:R -> R
- SW2: symbol chibi_2024-rescue:SW_PUSH_SMALL_H -> SW_PUSH_SMALL_H
- U1: symbol chibi_2024-rescue:LD1117S33CTR-RESCUE-chibi_2024 -> LD1117S33CTR
- U10: symbol components:74HCT125 -> 74HCT125
- U2: symbol chibi_2024-rescue:SP3485CN -> SP3485CN
- U3: symbol chibi_2024-rescue:STM32F030F4Px -> STM32F030F4Px
- U5, U7: symbol components:74HC595_mine -> 74HC595_mine
- Y1: symbol chibi_2024-rescue:Crystal_Small_5x3 -> Crystal_Small_5x3
Connections:
- net labels added: SEG_A_CTRL, SEG_B_CTRL, SEG_C_CTRL, SEG_DP_CTRL, SEG_D_CTRL, SEG_E_CTRL, SEG_F_CTRL, SEG_G_CTLR, WD_COMP1, WD_REF1, WD_REF2, in_left, in_right, ~WD_RST, ~WD_RST1, ~WD_RST2, ~WD_RSTQ
- net labels removed: SEGC0, SEGC1, SEGC2, SEGC3, SEGC4, SEGC5, SEGC6, SEGC7
- wire segments 211 -> 219
Other:
- moved on the sheet: P1, P3, Q1, Q2, Q3, Q4, Q5, Q6, Q7, Q8
