File: hw/chibi/layouttest/mux_module.sch (KiCad schematic (older format))
At the start: 7 parts, among them U9 MBI5026

Commit message: Add local changes
Parts:
- D14, D15, D16, D17: symbol components:7seg_4digit_cc -> 7seg_4digit_cc
- R38, R41: symbol chibi_2024-rescue:R -> R
- U9: symbol components:MBI5026 -> MBI5026
Connections:
- net at D14.12 (CC1): now also U9.17 (OUT12); no longer U9.6 (OUT1)
- net at D14.6 (CC4): now also U9.20 (OUT15); no longer U9.5 (OUT0)
- net at D14.8 (CC3): now also U9.19 (OUT14); no longer U9.11 (OUT6)
- net at D14.9 (CC2): now also U9.18 (OUT13); no longer U9.8 (OUT3)
- net at D15.12 (CC1): now also U9.13 (OUT8); no longer U9.7 (OUT2)
- net at D15.6 (CC4): now also U9.16 (OUT11); no longer U9.9 (OUT4)
- net at D15.8 (CC3): now also U9.15 (OUT10); no longer U9.10 (OUT5)
- net at D15.9 (CC2): now also U9.14 (OUT9); no longer U9.12 (OUT7)
- net at D16.12 (CC1): now also U9.9 (OUT4); no longer U9.14 (OUT9)
- net at D16.6 (CC4): now also U9.12 (OUT7); no longer U9.13 (OUT8)
- net at D16.8 (CC3): now also U9.11 (OUT6); no longer U9.16 (OUT11)
- net at D16.9 (CC2): now also U9.10 (OUT5); no longer U9.15 (OUT10)
- net at D17.12 (CC1): now also U9.5 (OUT0); no longer U9.18 (OUT13)
- net at D17.6 (CC4): now also U9.8 (OUT3); no longer U9.17 (OUT12)
- net at D17.8 (CC3): now also U9.7 (OUT2); no longer U9.20 (OUT15)
- net at D17.9 (CC2): now also U9.6 (OUT1); no longer U9.19 (OUT14)
Other:
- moved on the sheet: R40, R41
